File: kicad/CH340G_Programmer.kicad_sch (KiCad schematic)
At the start: 19 parts, among them J1 USB_B_Micro, J2 PROG, Q1 MMBT2222A 1P, Q2 MMBT2222A 1P, U1 AMS1117-3.3, U2 CH340G, Y1 12MHz

Commit message: Added jumper to allow choice of power to target or not.  Also added LED to indicate additional power rail
Parts:
- added D4: RED, LED_SMD:LED_0603_1608Metric, symbol Device:LED
- added JP?: PWR_TGT, Connector_PinHeader_2.54mm:PinHeader_1x02_P2.54mm_Vertical, symbol Jumper:Jumper_2_Bridged
- added R6: 330, Resistor_SMD:R_0603_1608Metric, symbol Device:R
Connections:
- net +3V3: now also JP?.1 (A), R6.1; no longer J2.1 (Pin_1), R3.1
- net GND: now also D4.1 (K)
- new net: D4.2 (A), R6.2
- new net: J2.1 (Pin_1), JP?.2 (B), R3.1
Other:
- moved on the sheet: D3, R3

Commit message: Corrected USB MicroB footprint to match the schematic - Was missing Pin6 (Shell)
Parts:
- gave numbers to parts that had none: 1
Changed lines of the file:
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@@
   (symbol (lib_id "power:+3V3") (at 223.52 91.44 0) (unit 1)
     (in_bom yes) (on_board yes) (fields_autoplaced)
-    (property "Reference" "#PWR?" (id 0) (at 223.52 95.25 0)
+    (property "Reference" "#PWR0102" (id 0) (at 223.52 95.25 0)
       (effects (font (size 1.27 1.27)) hide)
     )
@@
   (symbol (lib_id "Jumper:Jumper_2_Bridged") (at 228.6 91.44 0) (unit 1)
     (in_bom yes) (on_board yes)
-    (property "Reference" "JP?" (id 0) (at 228.6 85.09 0))
+    (property "Reference" "JP1" (id 0) (at 228.6 85.09 0))
     (property "Value" "PWR_TGT" (id 1) (at 228.6 87.63 0))
     (property "Footprint" "Connector_PinHeader_2.54mm:PinHeader_1x02_P2.54mm_Vertical" (id 2) (at 228.6 91.44 0)
@@
     )
     (path "/2c9e99d0-36de-47fd-8740-722bb7688943"
-      (reference "#PWR?") (unit 1) (value "+3V3") (footprint "")
+      (reference "#PWR0102") (unit 1) (value "+3V3") (footprint "")
     )
     (path "/ede17dd5-8d66-46f5-b58f-c99270bc800c"
@@
     )
     (path "/f5ca6e0b-35b7-4f19-9c39-537418dfc295"
-      (reference "JP?") (unit 1) (value "PWR_TGT") (footprint "Connector_PinHeader_2.54mm:PinHeader_1x02_P2.54mm_Vertical")
+      (reference "JP1") (unit 1) (value "PWR_TGT") (footprint "Connector_PinHeader_2.54mm:PinHeader_1x02_P2.54mm_Vertical")
     )
     (path "/290443a6-014d-4d23-88d9-9f3f579fa6c2"

Commit message: Added gerbers for last release
Parts:
- C1, C2, Q1, Q2, U1: JLCPCB_CORRECTION (none) -> 0; 0; 180
- J1, U2: JLCPCB_CORRECTION (none) -> 0; 0; 270
Other:
- note removed: "https://en.ovcharov.me/2019/08/16/ch340g-programmer-for-esp8266-esp32/"
Changed lines of the file:
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@@
     (stroke (width 0) (type default) (color 0 0 0 0))
-  )
-  (text "https://en.ovcharov.me/2019/08/16/ch340g-programmer-for-esp8266-esp32/"
-    (at 181.61 173.99 0)
-    (effects (font (size 1.27 1.27)) (justify left bottom))
   )
   (global_label "RXDI" (shape input) (at 247.65 151.13 270) (fields_autoplaced)
@@
       (effects (font (size 1.27 1.27)) hide)
     )
+    (property "JLCPCB_CORRECTION" "0; 0; 180" (id 5) (at 118.11 45.72 0)
+      (effects (font (size 1.27 1.27)) hide)
+    )
     (pin "1")
     (pin "2")
@@
       (effects (font (size 1.27 1.27)) hide)
     )
+    (property "JLCPCB_CORRECTION" "0; 0; 180" (id 5) (at 189.23 92.71 0)
+      (effects (font (size 1.27 1.27)) hide)
+    )
     (pin "1")
     (pin "2")
@@
     )
     (property "LCSC" "C8512" (id 4) (at 189.23 105.41 0)
+      (effects (font (size 1.27 1.27)) hide)
+    )
+    (property "JLCPCB_CORRECTION" "0; 0; 180" (id 5) (at 189.23 105.41 0)
       (effects (font (size 1.27 1.27)) hide)
     )
@@
     )
     (property "LCSC" "C319170" (id 4) (at 127 92.71 0)
+      (effects (font (size 1.27 1.27)) hide)
+    )
+    (property "JLCPCB_CORRECTION" "0; 0; 270" (id 5) (at 127 92.71 0)
       (effects (font (size 1.27 1.27)) hide)
     )
@@
     )
     (property "LCSC" "C14267" (id 4) (at 162.56 95.25 0)
+      (effects (font (size 1.27 1.27)) hide)
+    )
+    (property "JLCPCB_CORRECTION" "0; 0; 270" (id 5) (at 162.56 95.25 0)
       (effects (font (size 1.27 1.27)) hide)
     )
@@
       (effects (font (size 1.27 1.27)) hide)
     )
+    (property "JLCPCB_CORRECTION" "0; 0; 180" (id 5) (at 107.95 41.91 0)
+      (effects (font (size 1.27 1.27)) hide)
+    )
     (pin "1")
     (pin "2")
@@
       (effects (font (size 1.27 1.27)) hide)
     )
+    (property "JLCPCB_CORRECTION" "0; 0; 180" (id 5) (at 97.79 45.72 0)
+      (effects (font (size 1.27 1.27)) hide)
+    )
